Commit message: add : diff_drive.launch.py and meshes

File: urdf/model.urdf (robot description, URDF)
Before this commit: robot rover, 6 links, 5 joints
Joints:
- joint left_back_joint: origin xyz=-0.36808 0.37966 -0.16184 rpy=0 0 0 -> xyz=-0.38139 0.31387 -0.16074 rpy=0 0 0
- joint left_front_joint: origin xyz=0.3682 0.38012 -0.16177 rpy=0 0 0 -> xyz=0.38106 0.31837 -0.16074 rpy=0 0 0
- joint right_back_joint: origin xyz=-0.36808 -0.3807 -0.16164 rpy=0 0 0 -> xyz=-0.38139 -0.31387 -0.16074 rpy=0 0 0
- joint right_front_joint: origin xyz=0.3682 -0.37989 -0.16177 rpy=0 0 0 -> xyz=0.38106 -0.31837 -0.16074 rpy=0 0 0

File: urdf/model.urdf.xacro (robot description, xacro)
@@ -10,12 +10,27 @@
     <visual>
       <geometry>
-        <mesh filename="package://rover_sim/meshes/base_link.stl" />
-      </geometry>
-      <material name="grey"/>
-    </visual>
-    <collision>
-      <geometry>
-        <mesh filename="package://rover_sim/meshes/base_link.stl" />
-      </geometry>
+        <mesh filename="package://rover_sim/meshes/base_link.dae" />
+      </geometry>
+    </visual>
+    <collision>
+      <geometry>
+        <mesh filename="package://rover_sim/meshes/base_link.dae" />
+      </geometry>
+      <surface>
+        <friction>
+          <ode>
+            <mu>1.0</mu>          <!-- longitudinal friction -->
+            <mu2>1.0</mu2>        <!-- lateral friction -->
+            <slip1>0.0</slip1>    <!-- slip in longitudinal direction -->
+            <slip2>0.0</slip2>    <!-- slip in lateral direction -->
+          </ode>
+        </friction>
+        <contact>
+          <ode>
+            <kp>1e6</kp>          <!-- contact stiffness -->
+            <kd>1</kd>            <!-- contact damping -->
+          </ode>
+        </contact>
+      </surface>
     </collision>
     <inertial>
@@ -30,12 +45,28 @@
     <visual>
       <geometry>
-        <mesh filename="package://rover_sim/meshes/left_front.stl" />
-      </geometry>
-      <material name="pink"/>
-    </visual>
-    <collision>
-      <geometry>
-        <mesh filename="package://rover_sim/meshes/left_front.stl" />
-      </geometry>
+        <mesh filename="package://rover_sim/meshes/left_front.dae" />
+      </geometry>
+      <material name="pink"/>
+    </visual>
+    <collision>
+      <geometry>
+        <mesh filename="package://rover_sim/meshes/left_front.dae" />
+      </geometry>
+      <surface>
+        <friction>
+          <ode>
+            <mu>1.0</mu>          <!-- longitudinal friction -->
+            <mu2>1.0</mu2>        <!-- lateral friction -->
+            <slip1>0.0</slip1>    <!-- slip in longitudinal direction -->
+            <slip2>0.0</slip2>    <!-- slip in lateral direction -->
+          </ode>
+        </friction>
+        <contact>
+          <ode>
+            <kp>1e6</kp>          <!-- contact stiffness -->
+            <kd>1</kd>            <!-- contact damping -->
+          </ode>
+        </contact>
+      </surface>
     </collision>
     <inertial>
@@ -50,5 +81,5 @@
     <parent link="base_link" />
     <child link="left_front" />
-    <origin xyz="0.3682 0.38012 -0.16177" rpy="0 0 0" />
+    <origin xyz="0.38106 0.31837 -0.16074" rpy="0 0 0" />
     <axis xyz="0 1 0" />
   </joint>
@@ -56,12 +87,28 @@
     <visual>
       <geometry>
-        <mesh filename="package://rover_sim/meshes/right_front.stl" />
-      </geometry>
-      <material name="pink"/>
-    </visual>
-    <collision>
-      <geometry>
-        <mesh filename="package://rover_sim/meshes/right_front.stl" />
-      </geometry>
+        <mesh filename="package://rover_sim/meshes/right_front.dae" />
+      </geometry>
+      <material name="pink"/>
+    </visual>
+    <collision>
+      <geometry>
+        <mesh filename="package://rover_sim/meshes/right_front.dae" />
+      </geometry>
+      <surface>
+        <friction>
+          <ode>
+            <mu>1.0</mu>          <!-- longitudinal friction -->
+            <mu2>1.0</mu2>        <!-- lateral friction -->
+            <slip1>0.0</slip1>    <!-- slip in longitudinal direction -->
+            <slip2>0.0</slip2>    <!-- slip in lateral direction -->
+          </ode>
+        </friction>
+        <contact>
+          <ode>
+            <kp>1e6</kp>          <!-- contact stiffness -->
+            <kd>1</kd>            <!-- contact damping -->
+          </ode>
+        </contact>
+      </surface>
     </collision>
     <inertial>
@@ -76,5 +123,5 @@
     <parent link="base_link" />
     <child link="right_front" />
-    <origin xyz="0.3682 -0.37989 -0.16177" rpy="0 0 0" />
+    <origin xyz="0.38106 -0.31837 -0.16074" rpy="0 0 0" />
     <axis xyz="0 1 0" />
   </joint>
@@ -82,12 +129,28 @@
     <visual>
       <geometry>
-        <mesh filename="package://rover_sim/meshes/left_back.stl" />
-      </geometry>
-      <material name="pink"/>
-    </visual>
-    <collision>
-      <geometry>
-        <mesh filename="package://rover_sim/meshes/left_back.stl" />
-      </geometry>
+        <mesh filename="package://rover_sim/meshes/left_back.dae" />
+      </geometry>
+      <material name="pink"/>
+    </visual>
+    <collision>
+      <geometry>
+        <mesh filename="package://rover_sim/meshes/left_back.dae" />
+      </geometry>
+      <surface>
+        <friction>
+          <ode>
+            <mu>1.0</mu>          <!-- longitudinal friction -->
+            <mu2>1.0</mu2>        <!-- lateral friction -->
+            <slip1>0.0</slip1>    <!-- slip in longitudinal direction -->
+            <slip2>0.0</slip2>    <!-- slip in lateral direction -->
+          </ode>
+        </friction>
+        <contact>
+          <ode>
+            <kp>1e6</kp>          <!-- contact stiffness -->
+            <kd>1</kd>            <!-- contact damping -->
+          </ode>
+        </contact>
+      </surface>
     </collision>
     <inertial>
@@ -102,5 +165,5 @@
     <parent link="base_link" />
     <child link="left_back" />
-    <origin xyz="-0.36808 0.37966 -0.16184" rpy="0 0 0" />
+    <origin xyz="-0.38139 0.31387 -0.16074" rpy="0 0 0" />
     <axis xyz="0 1 0" />
   </joint>
@@ -108,12 +171,28 @@
     <visual>
       <geometry>
-        <mesh filename="package://rover_sim/meshes/right_back.stl" />
-      </geometry>
-      <material name="pink"/>
-    </visual>
-    <collision>
-      <geometry>
-        <mesh filename="package://rover_sim/meshes/right_back.stl" />
-      </geometry>
+        <mesh filename="package://rover_sim/meshes/right_back.dae" />
+      </geometry>
+      <material name="pink"/>
+    </visual>
+    <collision>
+      <geometry>
+        <mesh filename="package://rover_sim/meshes/right_back.dae" />
+      </geometry>
+      <surface>
+        <friction>
+          <ode>
+            <mu>1.0</mu>          <!-- longitudinal friction -->
+            <mu2>1.0</mu2>        <!-- lateral friction -->
+            <slip1>0.0</slip1>    <!-- slip in longitudinal direction -->
+            <slip2>0.0</slip2>    <!-- slip in lateral direction -->
+          </ode>
+        </friction>
+        <contact>
+          <ode>
+            <kp>1e6</kp>          <!-- contact stiffness -->
+            <kd>1</kd>            <!-- contact damping -->
+          </ode>
+        </contact>
+      </surface>
     </collision>
     <inertial>
@@ -128,5 +207,5 @@
     <parent link="base_link" />
     <child link="right_back" />
-    <origin xyz="-0.36808 -0.3807 -0.16164" rpy="0 0 0" />
+    <origin xyz="-0.38139 -0.31387 -0.16074" rpy="0 0 0" />
     <axis xyz="0 1 0" />
   </joint>
@@ -135,5 +214,5 @@
       <origin xyz="0 0 0" rpy="0 0 0" />
       <geometry>
-        <mesh filename="package://rover_sim/meshes/lidar.stl" />
+        <mesh filename="package://rover_sim/meshes/lidar.dae" />
       </geometry>
       <material name="pink" />
