Commit message: add : imu sensor

File: urdf/model.urdf.xacro (robot description, xacro)
@@ -72,8 +72,8 @@
     <inertial>
       <origin xyz="0.000053 0.04643 -0.000245" rpy="0 0 0" />
-      <mass value="1.80318326891779" />
-      <inertia ixx="0.0084266" ixy="0.0" ixz="0.0"
-             iyy="0.0141488" iyz="0.0"
-             izz="0.0084275"/>
+      <mass value="3.6" />
+      <inertia ixx="0.017" ixy="0.0" ixz="0.0"
+             iyy="0.028" iyz="0.0"
+             izz="0.017"/>
     </inertial>
   </link>
@@ -114,8 +114,8 @@
     <inertial>
       <origin xyz="-0.000053 -0.04643 -0.000245" rpy="0 0 0" />
-      <mass value="1.80318325796502" />
-      <inertia ixx="0.00841975" ixy="0.0" ixz="0.0"
-             iyy="0.01414883" iyz="0.0"
-             izz="0.00843434"/>
+      <mass value="3.6" />
+      <inertia ixx="0.017" ixy="0.0" ixz="0.0"
+             iyy="0.028" iyz="0.0"
+             izz="0.016"/>
     </inertial>
   </link>
@@ -156,8 +156,8 @@
     <inertial>
       <origin xyz="0.000053 0.04643 -0.000245" rpy="0 0 0" />
-      <mass value="1.80318324865192" />
-      <inertia ixx="0.00841984" ixy="0.0" ixz="0.0"
-             iyy="0.0141488" iyz="0.0"
-             izz="0.00843426"/>
+      <mass value="3.6" />
+      <inertia ixx="0.017" ixy="0.0" ixz="0.0"
+             iyy="0.028" iyz="0.0"
+             izz="0.017"/>
     </inertial>
   </link>
@@ -198,8 +198,8 @@
     <inertial>
       <origin xyz="-0.000053 -0.04643 -0.000245" rpy="0 0 0" />
-      <mass value="1.80318324711134" />
-      <inertia ixx="0.00841984" ixy="0.0" ixz="0.0"
-             iyy="0.01414883" iyz="0.0"
-             izz="0.00843426"/>
+      <mass value="3.6" />
+      <inertia ixx="0.017" ixy="0.0" ixz="0.0"
+             iyy="0.028" iyz="0.0"
+             izz="0.017"/>
     </inertial>
   </link>
@@ -224,4 +224,76 @@
     <origin xyz="0.2 0 0.20682" rpy="0 0 0"/>
   </joint>
+  <link name="imu">
+    <visual>
+      <origin xyz="0 0 0" rpy="0 0 0" />
+      <geometry>
+        <box size="0.03 0.02 0.01" />
+      </geometry>
+      <material name="pink" />
+    </visual>
+  </link>
+  <joint name='imu_joint' type='fixed'>
+    <parent link="base_link"/>
+    <child link="imu"/>
+    <origin xyz="0 0.05 0.03" rpy="0 0 0"/>
+  </joint>
+  <gazebo reference="imu">
+    <sensor type="imu" name="imu_sensor">
+      <always_on>true</always_on>
+      <update_rate>100</update_rate>   <!-- Hz -->
+      <visualize>true</visualize>
+      <imu>
+        <angular_velocity>
+            <x>
+              <noise type="gaussian">
+                <mean>0.0</mean>
+                <stddev>2e-4</stddev>
+              </noise>
+            </x>
+            <y>
+              <noise type="gaussian">
+                <mean>0.0</mean>
+                <stddev>2e-4</stddev>
+              </noise>
+            </y>
+            <z>
+              <noise type="gaussian">
+                <mean>0.0</mean>
+                <stddev>2e-4</stddev>
+              </noise>
+            </z>
+          </angular_velocity>
+          <linear_acceleration>
+            <x>
+              <noise type="gaussian">
+                <mean>0.0</mean>
+                <stddev>1.7e-2</stddev>
+              </noise>
+            </x>
+            <y>
+              <noise type="gaussian">
+                <mean>0.0</mean>
+                <stddev>1.7e-2</stddev>
+              </noise>
+            </y>
+            <z>
+              <noise type="gaussian">
+                <mean>0.0</mean>
+                <stddev>1.7e-2</stddev>
+              </noise>
+            </z>
+          </linear_acceleration>
+      </imu>
+      <plugin name="gazebo_ros_imu" filename="libgazebo_ros_imu_sensor.so">
+        <ros>
+          <namespace>/rover</namespace>
+          <remapping>~/out:=imu</remapping>
+        </ros>
+        <update_rate>100</update_rate>
+        <!-- <gaussian_noise>0.0001</gaussian_noise> --> <!-- remove other noises before uncommenting it> -->
+        <frame_name>imu</frame_name>
+      </plugin>
+    </sensor>
+  </gazebo>
   <gazebo reference="lidar">
     <sensor type="ray" name="laser">
