Commit message: add : camera urdf

File: urdf/camera.urdf.xacro (robot description, xacro)
@@ -210,5 +210,5 @@
     <axis xyz="0 1 0" />
   </joint>
-  <link name="lidar">
+  <link name="lidar_link">
     <visual>
       <origin xyz="0 0 0" rpy="0 0 0" />
@@ -221,8 +221,8 @@
   <joint name='lidar_joint' type='fixed'>
     <parent link="base_link"/>
-    <child link="lidar"/>
+    <child link="lidar_link"/>
     <origin xyz="0.2 0 0.20682" rpy="0 0 0"/>
   </joint>
-  <link name="imu">
+  <link name="imu_link">
     <visual>
       <origin xyz="0 0 0" rpy="0 0 0" />
@@ -235,8 +235,58 @@
   <joint name='imu_joint' type='fixed'>
     <parent link="base_link"/>
-    <child link="imu"/>
+    <child link="imu_link"/>
     <origin xyz="0 0.05 0.031" rpy="0 0 0"/>
   </joint>
-  <gazebo reference="imu">
+  <link name="camera_link">
+		<visual>
+			<geometry>
+				<box size="0.03 0.09 0.03"/>
+			</geometry>
+			<material name="camera_material">
+				<color rgba="0.3 0.3 0.3 1.0"/>
+			</material>
+		</visual>
+		<inertial>
+			<mass value="0.1"/>
+			<origin xyz="0 0 0" rpy="0 0 0"/>
+			<inertia ixx="1e-6" ixy="0" ixz="0" iyy="1e-6" iyz="0" izz="1e-6"/>
+		</inertial>
+	</link>
+	<joint name="camera_joint" type="fixed">
+		<parent link="base_link"/>
+		<child link="camera_link"/>
+		<origin xyz="0.28 0 0.12" rpy="0 0 0"/>
+	</joint>
+	<link name="camera_frame_link"></link>
+	<joint name="name" type="fixed">
+		<parent link="camera_link" />
+		<child link="camera_frame_link" />
+		<origin xyz="0 0 0" rpy="${-pi/2} 0 ${-pi/2}" />
+	</joint>
+	<gazebo reference="camera_link">
+		<sensor type="depth" name="camera">
+			<update_rate>5</update_rate>
+			<visualize>true</visualize>
+			<camera>
+				<horizontal_fov>1.5708</horizontal_fov>
+				<image>
+					<format>R8G8B8</format>
+					<width>640</width>
+					<height>480</height>
+				</image>
+				<clip>
+					<near>.05</near>
+					<far>20.0</far>
+				</clip>
+			</camera>
+			<plugin name="depth_camera" filename="libgazebo_ros_camera.so">
+				<ros>
+					<namespace>/rover</namespace>
+				</ros>
+				<frame_name>camera_frame_link</frame_name>
+			</plugin>
+		</sensor>
+	</gazebo>
+  <gazebo reference="imu_link">
     <sensor type="imu" name="imu_sensor">
       <always_on>true</always_on>
@@ -292,9 +342,9 @@
         <update_rate>100</update_rate>
         <!-- <gaussian_noise>0.0001</gaussian_noise> --> <!-- remove other noises before uncommenting it> -->
-        <frame_name>imu</frame_name>
+        <frame_name>imu_link</frame_name>
       </plugin>
     </sensor>
   </gazebo>
-  <gazebo reference="lidar">
+  <gazebo reference="lidar_link">
     <sensor type="ray" name="laser">
       <pose>0 0 0 0 0 0</pose>
@@ -322,5 +372,5 @@
         </ros>
         <output_type>sensor_msgs/LaserScan</output_type>
-        <frame_name>lidar</frame_name>
+        <frame_name>lidar_link</frame_name>
       </plugin>
     </sensor>

Commit message: add : rover_with_cam model

File: urdf/camera.urdf.xacro (robot description, xacro)
@@ -2,9 +2,12 @@
 <robot name="rover" xmlns:xacro="http://www.ros.org/wiki/xacro">
   <material name="grey">
-    <color rgba="0.4 0.4 0.4 1" />
+    <color rgba="0.4 0.4 0.45 1" />
   </material>
   <material name="pink">
     <color rgba="0.60 0.27 0.3 1" />
   </material>
+	<material name="light_green">
+		<color rgba="0.3 0.6 0.3 1"/>
+	</material>
   <link name="base_link">
     <visual>
@@ -230,5 +233,5 @@
         <box size="0.03 0.02 0.01" />
       </geometry>
-      <material name="pink" />
+      <material name="grey" />
     </visual>
   </link>
@@ -237,4 +240,18 @@
     <child link="imu_link"/>
     <origin xyz="0 0.05 0.031" rpy="0 0 0"/>
+  </joint>
+	<link name="gps_link">
+    <visual>
+      <origin xyz="0 0 0" rpy="0 0 0" />
+      <geometry>
+        <box size="0.03 0.02 0.01" />
+      </geometry>
+      <material name="light_green" />
+    </visual>
+  </link>
+	<joint name='gps_joint' type='fixed'>
+    <parent link="base_link"/>
+    <child link="gps_link"/>
+    <origin xyz="0 -0.05 0.031" rpy="0 0 0"/>
   </joint>
   <link name="camera_link">
@@ -288,8 +305,38 @@
 		</sensor>
 	</gazebo>
+	<gazebo reference="base_link">
+		<sensor name="gps" type="gps">
+			<always_on>true</always_on>
+			<update_rate>10</update_rate>
+			<visualize>true</visualize>
+			<gps>
+				<position_sensing>
+					<horizontal>
+						<noise type="gaussian">
+							<mean>0.0</mean>
+							<stddev>0.0002</stddev> <!-- ~20 cm noise -->
+						</noise>
+					</horizontal>
+					<vertical>
+						<noise type="gaussian">
+							<mean>0.0</mean>
+							<stddev>0.0004</stddev>
+						</noise>
+					</vertical>
+				</position_sensing>
+			</gps>
+			<plugin name="gps" filename="libgazebo_ros_gps_sensor.so">
+				<ros>
+					<namespace>/rover</namespace>
+					<remapping>fix:=gps/fix</remapping>
+				</ros>
+				<frame_id>gps_link</frame_id>
+			</plugin>
+		</sensor>
+	</gazebo>
   <gazebo reference="imu_link">
     <sensor type="imu" name="imu_sensor">
       <always_on>true</always_on>
-      <update_rate>100</update_rate>   <!-- Hz -->
+      <update_rate>100</update_rate>
       <visualize>true</visualize>
       <imu>
@@ -335,5 +382,5 @@
           </linear_acceleration>
       </imu>
-      <plugin name="gazebo_ros_imu" filename="libgazebo_ros_imu_sensor.so">
+      <plugin name="imu" filename="libgazebo_ros_imu_sensor.so">
         <ros>
           <namespace>/rover</namespace>
@@ -362,9 +409,9 @@
         <range>
           <min>0.1</min>
-          <max>2</max>
+          <max>15</max>
           <resolution>0.1</resolution>
         </range>
       </ray>
-      <plugin name="gazebo_ros_laser" filename="libgazebo_ros_ray_sensor.so">
+      <plugin name="laser" filename="libgazebo_ros_ray_sensor.so">
         <ros>
           <namespace>/rover</namespace>
@@ -377,5 +424,5 @@
   </gazebo>
   <gazebo>
-    <plugin name="rover_joint_state_publisher" filename="libgazebo_ros_joint_state_publisher.so">
+    <plugin name="joint_state_publisher" filename="libgazebo_ros_joint_state_publisher.so">
       <ros>
         <namespace>/rover</namespace>
