Commit message: fix: camera urdf and model

File: urdf/camera.urdf (robot description, URDF)
Before this commit: robot rover, 10 links, 9 joints
Joints:
- removed joint name
- added joint camera_link_joint: type fixed, parent camera_link, child camera_frame_link, origin xyz=0 0 0 rpy=-1.5707963267948966 0 -1.5707963267948966

File: urdf/camera.urdf.xacro (robot description, xacro)
@@ -276,5 +276,5 @@
 	</joint>
 	<link name="camera_frame_link"></link>
-	<joint name="name" type="fixed">
+	<joint name="camera_link_joint" type="fixed">
 		<parent link="camera_link" />
 		<child link="camera_frame_link" />
